File: Board/PWDTimer_8Lane/PWDTimer_8Lane.brd (EAGLE design)
At the start: 102.5 x 57.1 mm, 13 parts, among them J1 S3B-XH-A(LF)(SN), J2 S3B-XH-A(LF)(SN), J3 S3B-XH-A(LF)(SN), J4 S3B-XH-A(LF)(SN), J5 S3B-XH-A(LF)(SN), J6 S3B-XH-A(LF)(SN), J7 S3B-XH-A(LF)(SN), J8 S3B-XH-A(LF)(SN), P1 S2B-XH-A(LF)(SN), U1 ESP32-DEVKITC-32D

Commit message: Lots of updates to changing how data is stored as a json file, as well as starting the conversion to having groups and racers in the groups instead of just one monolothic racer group.
Parts:
- added J9: (no value), SparkFun-Connectors:1X19_NO_SILK
Connections:
- new net N$1: J9.4, U1.23
- new net N$10: J9.14, U1.33
- new net N$11: J9.15, U1.34
- new net N$12: J9.16, U1.35
- new net N$13: J9.17, U1.36
- new net N$14: J9.18, U1.37
- new net N$15: J9.19, U1.38
- new net N$2: J9.5, U1.24
- new net N$3: J9.6, U1.25
- new net N$4: J9.8, U1.27
- new net N$5: J9.9, U1.28
- new net N$6: J9.10, U1.29
- new net N$7: J9.11, U1.30
- new net N$8: J9.12, U1.31
- new net N$9: J9.13, U1.32
- net GATE: now also J9.3
- net GND: now also J9.1, J9.7
- net OUT8: now also J9.2
Routing:
- net N$9: track 0.00 -> 2.56 mm
- net N$5: track 0.00 -> 2.56 mm
- net N$12: track 0.00 -> 2.56 mm
- net N$15: track 0.00 -> 2.56 mm
- net N$8: track 0.00 -> 2.56 mm
- net N$14: track 0.00 -> 2.56 mm
- net N$13: track 0.00 -> 2.56 mm
- net N$11: track 0.00 -> 2.56 mm
- net N$10: track 0.00 -> 2.56 mm
- net N$7: track 0.00 -> 2.56 mm
- net N$6: track 0.00 -> 2.56 mm
- net N$4: track 0.00 -> 2.56 mm
- net N$3: track 0.00 -> 2.56 mm
- net N$2: track 0.00 -> 2.56 mm
- net N$1: track 0.00 -> 2.56 mm
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Other:
- board text added: "Two header rows allow for either 0.9in or 1.0in variants of the 38 pin ESP32 boards"
